Commit message: cellmap: Stage A plan-only — two-leg tag approach, collision-free, within limits
Captain decisions applied: tag 0 then tag 1; shoulder_pan +-120 deg
(confirmed); shoulder_link + upper_arm_link excluded from WORLD collision
only. That exclusion was the blocker — with it, planning against the
static map works.

Scoping of the collision fix is deliberately narrow. `collision:` and
`self_collision:` share one sphere set in the stock XRDF, so the
generator builds a separate world-only set that omits those two links and
leaves self_collision pointing at the FULL set. Verified in the output:
world set = forearm/wrist_1/2/3/tool0 (buffers 0.04), self set = all
seven links with the ignore rules intact.

find_standoff.py searches for a standoff configuration in JOINT space.
A Cartesian pose goal is the obvious approach and it does not work here:
with wrist_2 at +-30 deg and wrist_3 at +-20 deg the reachable
orientation family is narrow, so cuMotion returns
INVERSE_KINEMATICS_FAILURE for almost any full 6-DoF pose — which says
nothing about whether a good standoff exists. Searching joint space keeps
the windows satisfied by construction and scores on what matters: where
the camera ends up and whether it looks at the tag. Two traps found and
fixed inside it: a solution on a window EDGE is rejected by cuMotion as
'exceeds limits' (floating point puts it a fraction outside), hence
--inset-deg; and without a height floor the search returns a pose 12 cm
above the table that is geometrically close but in collision.

Joint limits are clamped to the mechanical range: +-120 deg around a pan
of -246.8 deg reaches -366.8, outside the UR10's +-360, and a URDF that
claims more travel than the robot has is worse than the wide limits we
started from.

show_plan.py publishes saved plans as markers on /cellmap/plan_path
(transient-local so a late RViz still sees them) and cellmap.rviz gains
the display, so the captain can watch the path against the map.

Result, PLAN ONLY, nothing executed:
  leg 1  current -> tag0 standoff  202 pts, 20.1 s, 1.800 m (1.22x)
  leg 2  tag0 -> tag1 standoff      54 pts,  5.3 s, 0.484 m (1.02x)
  tool0 stays 31.7-76.9 cm above the table; closest approach to either
  tag 32.1 cm; every waypoint inside the windows, tightest margin
  shoulder_pan 2.0 deg.

Co-Authored-By: Claude Opus 5 <noreply@anthropic.com>
Claude-Session: https://claude.ai/code/session_01BiUDeE4zksLtZ8BqQipr4n

File: cumotion/ur10_pneumatic.urdf (robot description, URDF)
Before this commit: robot ur10, 13 links, 12 joints
Joints:
- joint elbow_joint: limit lower=0.782215 upper=2.353011 effort=150.0 velocity=3.141592653589793 -> lower=0.782167 upper=2.352963 effort=150.0 velocity=3.141592653589793
- joint shoulder_lift_joint: limit lower=-2.119050 upper=-0.548254 effort=330.0 velocity=2.0943951023931953 -> lower=-2.119158 upper=-0.548362 effort=330.0 velocity=2.0943951023931953
- joint shoulder_pan_joint: limit lower=-4.830280 upper=-3.783083 effort=330.0 velocity=2.0943951023931953 -> lower=-6.283185 upper=-2.213223 effort=330.0 velocity=2.0943951023931953
- joint wrist_1_joint: limit lower=2.153186 upper=3.723982 effort=56.0 velocity=3.141592653589793 -> lower=2.153162 upper=3.723959 effort=56.0 velocity=3.141592653589793
- joint wrist_2_joint: limit lower=3.843378 upper=4.890576 effort=56.0 velocity=3.141592653589793 -> lower=3.843390 upper=4.890588 effort=56.0 velocity=3.141592653589793
