Commit message: cumotion: captain-declared shoulder_lift override + full-world-collision limited model (Phase C)
Phase C of the measured-limits task. Adds the declared-override mechanism the
captain's 2026-09-04 decision needs, applies it, and regenerates the limited
model against the cleaned map — but the tag1->shelf re-plan within these limits
is BLOCKED and escalated (see below).

- record_joint_limits.py: new --declare JOINT=MIN,MAX --reason mode (no rig, no
  recording). Widens ONE joint in the existing measured file to
  [MIN-slack, MAX+slack] deg to COVER a known-required travel the hand-sweep did
  not reach, recorded under a separate top-level `declared:` block
  (source=captain-declared, NOT hand-swept) so provenance stays unambiguous
  (5 measured, 1 declared). Every other joint stays byte-identical; the joint's
  own measured.extremes_* are left as measured. Idempotent per joint.
- make_limited_urdf.py: new --keep-world-collision flag. Keeps the FULL collision
  sphere set for WORLD collision (does not drop shoulder_link/upper_arm_link) —
  correct against a CLEANED map that no longer carries the mounting pedestal the
  exclusion existed for. Retract config is still moved inside the windows.
- measured_joint_limits.yaml: shoulder_lift declared to cover the validated demo
  travel [-174.17, -12.23] +-1 deg slack -> window [-175.17, -11.23] deg
  (extended from measured raw -173.8..-97.2 by captain instruction). Other 5
  joints unchanged.
- ur10_measured.urdf/.xrdf: regenerated (--frozen --keep-world-collision).
- Tests: +6 (declare widen/refuse/idempotent, execute_plan + make_limited_urdf
  round-trips of a declared file, keep-world-collision). 18/18 offline, no rig.

Phase C re-plan BLOCKED (needs-decision): with the measured+declared limits the
cuMotion re-plan of tag1->shelf FAILS (INVERSE_KINEMATICS_FAILURE). The demo also
needs elbow -61.7 (win floor -47.8; raw sweep -52.8), wrist_1 355.1 (win 348.2;
raw physical bind 353.2 — 1.9 deg PAST the hand-swept stop) and wrist_2 -82.4
(win -76.0; raw -81.0) outside their MEASURED windows. The one in-window goal IK
is a different elbow-up posture unreachable without a 177 deg wrist_1 rewind
(> 170 deg guard). Not loosening limits unilaterally.

Co-Authored-By: Claude Opus 4.8 <noreply@anthropic.com>
Claude-Session: https://claude.ai/code/session_01CjZa1ZTsrDRRjcog2da3WF

File: cumotion/ur10_measured.urdf (robot description, URDF)
Before this commit: robot ur10, 13 links, 12 joints
Joints:
- joint shoulder_lift_joint: limit lower=-2.946110 upper=-1.783860 effort=330.0 velocity=2.0943951023931953 -> lower=-3.057365 upper=-0.196061 effort=330.0 velocity=2.0943951023931953

Commit message: cumotion: tag1->shelf re-validated within measured+declared limits; executable plan + note
Completes Phase C. The captain accepted extending the measured limits by the
minimum the tag1->shelf route needs (decision 2026-09-05). Applied, re-planned,
validated, and delivered the executable plan + captain command. Plan-only; no arm
motion.

- record_joint_limits.py --declare: now UNION semantics (only ever widens the
  side the required travel needs, keeps the measured bound on the other side), so
  a one-sided floor extension can't collapse a joint's ceiling. Records
  prior_window_deg in the declared entry. +2 tests (one-sided keep, only-widens);
  20/20 offline, no rig.
- measured_joint_limits.yaml: three captain-declared windows now — shoulder_lift
  [-175.2,-11.2] (both ends), elbow floor -62.7, wrist_2 floor -83.4 (one-sided;
  measured ceilings kept). wrist_1 stays MEASURED [162.8,348.2] and was NOT
  extended: the re-plan routes wrist_1 <= 339.77 (inside measured), so nothing is
  declared past the hand-swept physical bind. Other joints byte-identical measured.
- ur10_measured.urdf/.xrdf regenerated (--frozen --keep-world-collision -> full
  world collision on the cleaned map; explicit outputs, pneumatic defaults
  untouched).
- plans/tag1-shelf-measlim.yaml: fresh cuMotion re-plan (committed start, same
  shelf standoff pose), 276 pts, error_code 1, every waypoint inside the
  measured+declared windows (tightest 1.0 deg), max joint delta 161.9<170. Box
  sweeps clear: table +4.8 cm, shelf +13.7 cm. execute_plan --limits dry-check
  passes (exact-mode peak vel 5.0%). Evidence:
  plan-measlim-clearance-checks.md, render plan-measlim-vs-cumotion.png.
- captain-execute-note.md: now the DEFINITIVE executable note — exact single
  command (execute_plan.py --exact --limits cumotion/measured_joint_limits.yaml),
  prerequisites (incl. frozen-feed recovery + tray-detector restart + planner
  from a live copy), safety checklist, and a plain-English disclosure of every
  declared extension (measured raw vs declared, why).
- RUNBOOK sec 10: measured-vs-declared limits pointer and how to re-measure /
  re-declare when the line is re-routed or the arm re-parked.

Supersedes for execution the collision-evidence plan tag1-shelf-cumotion.yaml
(drove wrist_1 to 355.1, past the 353.2 bind).

Co-Authored-By: Claude Opus 4.8 <noreply@anthropic.com>
Claude-Session: https://claude.ai/code/session_01CjZa1ZTsrDRRjcog2da3WF

File: cumotion/ur10_measured.urdf (robot description, URDF)
Before this commit: robot ur10, 13 links, 12 joints
Joints:
- joint elbow_joint: limit lower=-0.833770 upper=1.906338 effort=150.0 velocity=3.141592653589793 -> lower=-1.093788 upper=1.906338 effort=150.0 velocity=3.141592653589793
- joint wrist_2_joint: limit lower=-1.326520 upper=2.013530 effort=56.0 velocity=3.141592653589793 -> lower=-1.454848 upper=2.013530 effort=56.0 velocity=3.141592653589793
